File: Kicad/PowerPole.sch (KiCad schematic (older format))
At the start: 41 parts, among them J1 Anderson powerpole, J2 Anderson powerpole, J3 Anderson powerpole, J4 Anderson powerpole, J5 Anderson powerpole, K1 896HP-1AH-C-12VDC, SW1 SW_Push

Commit message: PCB update
Parts:
- added J6: Meter +ve, Connector_Wire:SolderWire-0.5sqmm_1x01_D0.9mm_OD2.1mm, symbol Connector:Screw_Terminal_01x01
- added J7: Meter GND, Connector_Wire:SolderWire-2.5sqmm_1x01_D2.4mm_OD4.4mm, symbol Connector:Screw_Terminal_01x01
- added J8: Meter LOAD, Connector_Wire:SolderWire-2.5sqmm_1x01_D2.4mm_OD4.4mm, symbol Connector:Screw_Terminal_01x01
Connections:
- net Vout: now reaches D1.2 (A), D12.2 (A), D2.2 (A), D3.1 (K), D4.1 (A1), D5.1 (A1), F2.3, F2.4, F3.3, F3.4, F4.3, F4.4, F5.3, F5.4, K1.87 (NO), R3.1
- net GND: now reaches C1.2, C2.2, C3.2, C4.2, C5.2, D1.1 (K), D10.1 (K), D13.2 (A), D15.1 (K), D2.1 (K), D4.2 (A2), D5.2 (A2), D6.1 (K), D7.1 (K), D8.1 (K), D9.1 (K), J2.2 (-ve), J3.2 (-ve), J4.2 (-ve), J5.2 (-ve), K1.85 (COIL_1), R1.2
- net GND: now also J8.1 (Pin_1); no longer J1.2 (-ve)
- net at D14.2 (A), F1.3, F1.4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: now also J6.1 (Pin_1)
- new net: J1.2 (-ve), J7.1 (Pin_1)

Commit message: Fixed value of led resistors
Parts:
- R3, R4, R5, R6, R7, R8: value 220K -> 2K2
Changed lines of the file:
@@
 P 4500 2650
 F 0 "R3" H 4570 2696 50  0000 L CNN
-F 1 "220K" H 4570 2605 50  0000 L CNN
+F 1 "2K2" H 4570 2605 50  0000 L CNN
 F 2 "Resistor_THT:R_Axial_DIN0207_L6.3mm_D2.5mm_P10.16mm_Horizontal" V 4430 2650 50  0001 C CNN
 F 3 "~" H 4500 2650 50  0001 C CNN
@@
 P 7950 4200
 F 0 "R4" V 7743 4200 50  0000 C CNN
-F 1 "220K" V 7834 4200 50  0000 C CNN
+F 1 "2K2" V 7834 4200 50  0000 C CNN
 F 2 "Resistor_THT:R_Axial_DIN0207_L6.3mm_D2.5mm_P10.16mm_Horizontal" V 7880 4200 50  0001 C CNN
 F 3 "~" H 7950 4200 50  0001 C CNN
@@
 P 7050 4200
 F 0 "R5" V 6843 4200 50  0000 C CNN
-F 1 "220K" V 6934 4200 50  0000 C CNN
+F 1 "2K2" V 6934 4200 50  0000 C CNN
 F 2 "Resistor_THT:R_Axial_DIN0207_L6.3mm_D2.5mm_P10.16mm_Horizontal" V 6980 4200 50  0001 C CNN
 F 3 "~" H 7050 4200 50  0001 C CNN
@@
 P 6100 4200
 F 0 "R6" V 5893 4200 50  0000 C CNN
-F 1 "220K" V 5984 4200 50  0000 C CNN
+F 1 "2K2" V 5984 4200 50  0000 C CNN
 F 2 "Resistor_THT:R_Axial_DIN0207_L6.3mm_D2.5mm_P10.16mm_Horizontal" V 6030 4200 50  0001 C CNN
 F 3 "~" H 6100 4200 50  0001 C CNN
@@
 P 5200 4200
 F 0 "R7" V 4993 4200 50  0000 C CNN
-F 1 "220K" V 5084 4200 50  0000 C CNN
+F 1 "2K2" V 5084 4200 50  0000 C CNN
 F 2 "Resistor_THT:R_Axial_DIN0207_L6.3mm_D2.5mm_P10.16mm_Horizontal" V 5130 4200 50  0001 C CNN
 F 3 "~" H 5200 4200 50  0001 C CNN
@@
 P 2300 2750
 F 0 "R8" H 2370 2796 50  0000 L CNN
-F 1 "220K" H 2370 2705 50  0000 L CNN
+F 1 "2K2" H 2370 2705 50  0000 L CNN
 F 2 "Resistor_THT:R_Axial_DIN0207_L6.3mm_D2.5mm_P10.16mm_Horizontal" V 2230 2750 50  0001 C CNN
 F 3 "~" H 2300 2750 50  0001 C CNN

Commit message: Updated to v1.1. powerpole sinkscreen and sw1 pads updated
Parts:
- SW1: footprint Connector_Wire:SolderWire-0.1sqmm_1x02_P3.6mm_D0.4mm_OD1mm -> Connector_Wire:SolderWire-0.25sqmm_1x02_P4.2mm_D0.65mm_OD1.7mm
Changed lines of the file:
@@
 F 0 "SW1" H 3400 2185 50  0000 C CNN
 F 1 "SW_Push" H 3400 2094 50  0000 C CNN
-F 2 "Connector_Wire:SolderWire-0.1sqmm_1x02_P3.6mm_D0.4mm_OD1mm" H 3400 2100 50  0001 C CNN
+F 2 "Connector_Wire:SolderWire-0.25sqmm_1x02_P4.2mm_D0.65mm_OD1.7mm" H 3400 2100 50  0001 C CNN
 F 3 "~" H 3400 2100 50  0001 C CNN
 	1    3400 1900
